File: Circuit Diagram/Circuit Diagram.kicad_sch (KiCad schematic)
At the start: 3 parts, among them M1 Motor_Servo, M2 Motor_Servo

Commit message: update
Parts:
- added M3: Motor_Servo, symbol Motor:Motor_Servo
- added M4: Stepper_Motor_bipolar, symbol Motor:Stepper_Motor_bipolar
- added U1: ULN2003A, symbol Transistor_Array:ULN2003A
Connections:
- net +5V: now also M3.2 (+), U1.9 (COM)
- net GND: now also A1.29 (GND), M3.3 (-), U1.8 (GND)
- net at A1.17 (D2): now also U1.1 (I1)
- net at A1.19 (D4): now also U1.2 (I2)
- net at A1.22 (D7): now also U1.3 (I3)
- net at A1.23 (D8): now also U1.4 (I4)
- net at A1.25 (D10): now also M3.1 (PWM); no longer M2.1 (PWM)
- net at M1.1 (PWM): now also A1.27 (D12); no longer A1.26 (D11)
- new net: M4.2 (-), U1.13 (O4)
- new net: M4.1, U1.14 (O3)
- new net: M4.3, U1.15 (O2)
- new net: M4.4, U1.16 (O1)
- new net: A1.26 (D11), M2.1 (PWM)
Other:
- company: (none) -> Zenith Harmonics
- title: (none) -> GELU - Circuit Diagram
- moved on the sheet: A1
